File: MCB19/supplies.sch (KiCad schematic (older format))
At the start: 6 parts, among them U501 LM7805

Commit message: New version
Detalhes
Parts:
- U301: renamed from U501; value LM7805 -> LM7815
- renumbered C501 to C301, C502 to C302, C503 to C303, C504 to C304, D501 to D301
Connections:
- net +5V_OUT renamed +15V_OUT
Changed lines of the file:
@@
 $Descr A4 11693 8268
 encoding utf-8
-Sheet 3 6
+Sheet 3 7
 Title ""
 Date ""
@@
 $EndDescr
 $Comp
-L Regulator_Linear:LM7805_TO220 U501
+L Regulator_Linear:LM7805_TO220 U301
 U 1 1 5A007B62
 P 5900 3950
-F 0 "U501" H 5750 4075 50  0000 C CNN
-F 1 "LM7805" H 5900 4100 50  0000 L CNN
+AR Path="/5AACFFEF/5A007B62" Ref="U301"  Part="1"
+AR Path="/5D9BEA13/5A007B62" Ref="U301"  Part="1"
+F 0 "U301" H 5750 4075 50  0000 C CNN
+F 1 "LM7815" H 5900 4100 50  0000 L CNN
 F 2 "KicadZeniteSolarLibrary18:TO-220-3_Horizontal_TabDown_SMD" H 5900 4175 50  0001 C CIN
 F 3 "https://www.sparkfun.com/datasheets/Components/LM7805.pdf" H 5900 3900 50  0001 C CNN
@@
 GND
 Text HLabel 6650 3750 2    60   Input ~ 0
-+5V_OUT
++15V_OUT
 $Comp
-L Device:CP1_Small C501
+L Device:CP1_Small C301
 U 1 1 5A008895
 P 4900 4400
-F 0 "C501" H 4910 4470 50  0000 L CNN
+AR Path="/5AACFFEF/5A008895" Ref="C301"  Part="1"
+AR Path="/5D9BEA13/5A008895" Ref="C301"  Part="1"
+F 0 "C301" H 4910 4470 50  0000 L CNN
 F 1 "1uF" H 4910 4320 50  0000 L CNN
 F 2 "Capacitor_Tantalum_SMD:CP_EIA-6032-20_AVX-F_Pad2.25x2.35mm_HandSolder" H 4900 4400 50  0001 C CNN
@@
 $EndComp
 $Comp
-L Device:C_Small C502
+L Device:C_Small C302
 U 1 1 5A00899A
 P 5200 4400
-F 0 "C502" H 5210 4470 50  0000 L CNN
+AR Path="/5AACFFEF/5A00899A" Ref="C302"  Part="1"
+AR Path="/5D9BEA13/5A00899A" Ref="C301"  Part="1"
+F 0 "C302" H 5210 4470 50  0000 L CNN
 F 1 "100nF" H 5210 4320 50  0000 L CNN
 F 2 "Capacitor_SMD:C_0805_2012Metric_Pad1.15x1.40mm_HandSolder" H 5200 4400 50  0001 C CNN
@@
 +18V_IN
 $Comp
-L Device:C_Small C503
+L Device:C_Small C303
 U 1 1 5A00B18A
 P 6500 4400
-F 0 "C503" H 6510 4470 50  0000 L CNN
+AR Path="/5AACFFEF/5A00B18A" Ref="C303"  Part="1"
+AR Path="/5D9BEA13/5A00B18A" Ref="C303"  Part="1"
+F 0 "C303" H 6510 4470 50  0000 L CNN
 F 1 "100nF" H 6510 4320 50  0000 L CNN
 F 2 "Capacitor_SMD:C_0805_2012Metric_Pad1.15x1.40mm_HandSolder" H 6500 4400 50  0001 C CNN
@@
 $EndComp
 $Comp
-L Device:CP1_Small C504
+L Device:CP1_Small C304
 U 1 1 5AAD0D5C
 P 6850 4400
-F 0 "C504" H 6860 4470 50  0000 L CNN
+AR Path="/5AACFFEF/5AAD0D5C" Ref="C304"  Part="1"
+AR Path="/5D9BEA13/5AAD0D5C" Ref="C304"  Part="1"
+F 0 "C304" H 6860 4470 50  0000 L CNN
 F 1 "1uF" H 6860 4320 50  0000 L CNN
 F 2 "Capacitor_Tantalum_SMD:CP_EIA-6032-20_AVX-F_Pad2.25x2.35mm_HandSolder" H 6850 4400 50  0001 C CNN
@@
 U 1 1 5BE75359
 P 5200 3450
+AR Path="/5AACFFEF/5BE75359" Ref="#FLG0501"  Part="1"
+AR Path="/5D9BEA13/5BE75359" Ref="#FLG0101"  Part="1"
 F 0 "#FLG0501" H 5200 3525 50  0001 C CNN
 F 1 "PWR_FLAG" H 5200 3650 50  0000 C CNN
@@
 U 1 1 5BE753AF
 P 5200 4900
+AR Path="/5AACFFEF/5BE753AF" Ref="#FLG0502"  Part="1"
+AR Path="/5D9BEA13/5BE753AF" Ref="#FLG0102"  Part="1"
 F 0 "#FLG0502" H 5200 4975 50  0001 C CNN
 F 1 "PWR_FLAG" H 5200 5100 50  0000 C CNN
@@
 	5200 3450 5200 3950
 $Comp
-L Diode:LL4148 D501
+L Diode:LL4148 D301
 U 1 1 5A009BD5
 P 4675 3950
-F 0 "D501" H 4675 4050 50  0000 C CNN
+AR Path="/5AACFFEF/5A009BD5" Ref="D301"  Part="1"
+AR Path="/5D9BEA13/5A009BD5" Ref="D301"  Part="1"
+F 0 "D301" H 4675 4050 50  0000 C CNN
 F 1 "LL4148" H 4675 3850 50  0000 C CNN
 F 2 "Diode_SMD:D_MiniMELF_Handsoldering" H 4675 3775 50  0001 C CNN

Commit message: Versão 2.0
Novas modificações, após confirmado, pode ser fabricada
Parts:
- U301: value LM7815 -> LM7805
Connections:
- net +15V_OUT renamed +5V_OUT
Changed lines of the file:
@@
 AR Path="/5D9BEA13/5A007B62" Ref="U301"  Part="1"
 F 0 "U301" H 5750 4075 50  0000 C CNN
-F 1 "LM7815" H 5900 4100 50  0000 L CNN
+F 1 "LM7805" H 5900 4100 50  0000 L CNN
 F 2 "KicadZeniteSolarLibrary18:TO-220-3_Horizontal_TabDown_SMD" H 5900 4175 50  0001 C CIN
 F 3 "https://www.sparkfun.com/datasheets/Components/LM7805.pdf" H 5900 3900 50  0001 C CNN
@@
 GND
 Text HLabel 6650 3750 2    60   Input ~ 0
-+15V_OUT
++5V_OUT
 $Comp
 L Device:CP1_Small C301
