File: hardware/canbus.sch (KiCad schematic (older format))
At the start: 21 parts, among them U201 MCP2551-I/SN, U202 MCP2515-xSO, Y201 16MHz

Commit message: Some fixes, ready for heat transfering
Parts:
- R201: value 120 -> 1k
Changed lines of the file:
@@
 P 8200 3600
 F 0 "R201" V 8050 3550 50  0000 L CNN
-F 1 "120" V 8100 3550 50  0000 L CNN
+F 1 "1k" V 8100 3550 50  0000 L CNN
 F 2 "Resistor_SMD:R_0805_2012Metric_Pad1.15x1.40mm_HandSolder" H 8200 3600 50  0001 C CNN
 F 3 "" H 8200 3600 50  0001 C CNN
