File: hardware/driver.sch (KiCad schematic (older format))
At the start: 51 parts, among them J611 +BAT_IN, J612 -BAT_IN, J613 +BAT_OUT, J614 -BAT_OUT, Q601 IRFP260N, Q602 IRFP260N, U601 LM5104MNOPB, U602 INA240A4D, U603 LM324

Commit message: enable, vi, vo
Parts:
- added Q603: BC857, Package_TO_SOT_SMD:SOT-23, symbol Transistor_BJT:BC857
- added Q604: BC847, Package_TO_SOT_SMD:SOT-23, symbol Transistor_BJT:BC847
- added R611, R612: 1k, Resistor_SMD:R_0805_2012Metric_Pad1.15x1.40mm_HandSolder, symbol Device:R_Small
- added R?: 15k, Resistor_SMD:R_0805_2012Metric_Pad1.15x1.40mm_HandSolder, symbol Device:R_Small
- added R?: 1k2, Resistor_SMD:R_0805_2012Metric_Pad1.15x1.40mm_HandSolder, symbol Device:R_Small
- R609: value 470R -> 15k
- R610: value 1k5 -> 1k2
- gave numbers to parts that had none: 1
Connections:
- net labels added: enable
- wire segments 193 -> 207
Other:
- moved on the sheet: C604, C605, C612, F601, J612, J614, R609, R610, U603A, U603E

Commit message: Adição das mudanças pré-DSB(SF) feitas no MCB19
Parts:
- gave numbers to parts that had none: 2
Connections:
- net labels added: ENABLE, LM324B
- net labels removed: enable
- wire segments 207 -> 216
Other:
- moved on the sheet: U603B, U603D
Changed lines of the file:
@@
 EESchema Schematic File Version 4
-EELAYER 30 0
+EELAYER 26 0
 EELAYER END
 $Descr A4 11693 8268
@@
 $Comp
 L Amplifier_Operational:LM324 U603
-U 2 1 5D47935F
-P 6875 4625
-F 0 "U603" H 6875 4992 50  0000 C CNN
-F 1 "LM324" H 6875 4901 50  0000 C CNN
-F 2 "Package_SO:SOIC-14_3.9x8.7mm_P1.27mm" H 6825 4725 50  0001 C CNN
-F 3 "http://www.ti.com/lit/ds/symlink/lm2902-n.pdf" H 6925 4825 50  0001 C CNN
-	2    6875 4625
-	1    0    0    -1
-$EndComp
-$Comp
-L Amplifier_Operational:LM324 U603
 U 3 1 5D4793F4
 P 7575 4625
@@
 L Amplifier_Operational:LM324 U603
 U 4 1 5D479479
-P 6175 4625
-F 0 "U603" H 6175 4992 50  0000 C CNN
-F 1 "LM324" H 6175 4901 50  0000 C CNN
-F 2 "Package_SO:SOIC-14_3.9x8.7mm_P1.27mm" H 6125 4725 50  0001 C CNN
-F 3 "http://www.ti.com/lit/ds/symlink/lm2902-n.pdf" H 6225 4825 50  0001 C CNN
-	4    6175 4625
+P 8375 4625
+F 0 "U603" H 8375 4992 50  0000 C CNN
+F 1 "LM324" H 8375 4901 50  0000 C CNN
+F 2 "Package_SO:SOIC-14_3.9x8.7mm_P1.27mm" H 8325 4725 50  0001 C CNN
+F 3 "http://www.ti.com/lit/ds/symlink/lm2902-n.pdf" H 8425 4825 50  0001 C CNN
+	4    8375 4625
 	1    0    0    -1
 $EndComp
@@
 	7250 4725 7275 4725
 Wire Wire Line
-	6575 4525 6550 4525
-Wire Wire Line
-	6550 4525 6550 4725
-Wire Wire Line
-	6550 4725 6575 4725
-Wire Wire Line
-	5875 4525 5850 4525
-Wire Wire Line
-	5850 4525 5850 4725
-Wire Wire Line
-	5850 4725 5875 4725
+	8075 4525 8050 4525
+Wire Wire Line
+	8050 4525 8050 4725
+Wire Wire Line
+	8050 4725 8075 4725
 $Comp
 L power:GND #PWR0610
 U 1 1 5D482B0D
-P 6475 4650
-F 0 "#PWR0610" H 6475 4400 50  0001 C CNN
-F 1 "GND" H 6480 4477 50  0000 C CNN
-F 2 "" H 6475 4650 50  0001 C CNN
-F 3 "" H 6475 4650 50  0001 C CNN
-	1    6475 4650
-	1    0    0    -1
-$EndComp
-$Comp
-L power:GND #PWR0611
-U 1 1 5D482F12
-P 7175 4650
-F 0 "#PWR0611" H 7175 4400 50  0001 C CNN
-F 1 "GND" H 7180 4477 50  0000 C CNN
-F 2 "" H 7175 4650 50  0001 C CNN
-F 3 "" H 7175 4650 50  0001 C CNN
-	1    7175 4650
+P 8675 4650
+F 0 "#PWR0610" H 8675 4400 50  0001 C CNN
+F 1 "GND" H 8680 4477 50  0000 C CNN
+F 2 "" H 8675 4650 50  0001 C CNN
+F 3 "" H 8675 4650 50  0001 C CNN
+	1    8675 4650
 	1    0    0    -1
 $EndComp
@@
 	7875 4625 7875 4650
 Wire Wire Line
-	7175 4625 7175 4650
-Wire Wire Line
-	6475 4625 6475 4650
+	8675 4625 8675 4650
 $Comp
 L power:+5V #PWR0608
@@
 LM324A
 Wire Wire Line
-	9100 1900 9025 1900
+	9100 1900 9050 1900
 Wire Wire Line
 	5875 1900 5900 1900
@@
 $EndComp
 Text HLabel 1300 3450 0    50   Input ~ 0
-enable
+ENABLE
 $Comp
 L power:GND #PWR0616
@@
 	7500 3950 7800 3950
 $Comp
-L Device:R_Small R?
+L Device:R_Small R613
 U 1 1 5E2900F5
 P 4250 3225
-F 0 "R?" V 4150 3225 50  0000 C CNN
+F 0 "R613" V 4150 3225 50  0000 C CNN
 F 1 "15k" V 4075 3225 50  0000 C CNN
 F 2 "Resistor_SMD:R_0805_2012Metric_Pad1.15x1.40mm_HandSolder" H 4250 3225 50  0001 C CNN
@@
 $EndComp
 $Comp
-L Device:R_Small R?
+L Device:R_Small R614
 U 1 1 5E2900FF
 P 4250 3525
-F 0 "R?" V 4325 3525 50  0000 C CNN
+F 0 "R614" V 4325 3525 50  0000 C CNN
 F 1 "1k2" V 4400 3525 50  0000 C CNN
 F 2 "Resistor_SMD:R_0805_2012Metric_Pad1.15x1.40mm_HandSolder" H 4250 3525 50  0001 C CNN
@@
 Wire Wire Line
 	4250 3950 4525 3950
-Wire Wire Line
-	4350 3375 4350 1925
-Wire Wire Line
-	7600 3650 7600 1925
+$Comp
+L Amplifier_Operational:LM324 U603
+U 2 1 5D47935F
+P 4775 1900
+F 0 "U603" H 4775 2267 50  0000 C CNN
+F 1 "LM324" H 4775 2176 50  0000 C CNN
+F 2 "Package_SO:SOIC-14_3.9x8.7mm_P1.27mm" H 4725 2000 50  0001 C CNN
+F 3 "http://www.ti.com/lit/ds/symlink/lm2902-n.pdf" H 4825 2100 50  0001 C CNN
+	2    4775 1900
+	1    0    0    -1
+$EndComp
+Wire Wire Line
+	4475 1800 4350 1800
+Wire Wire Line
+	4350 1800 4350 3375
+Wire Wire Line
+	4475 2000 4450 2000
+Wire Wire Line
+	4450 2000 4450 2125
+Wire Wire Line
+	4450 2125 5100 2125
+Wire Wire Line
+	5100 2125 5100 1900
+Wire Wire Line
+	5100 1900 5075 1900
+Wire Wire Line
+	8425 1800 7600 1800
+Wire Wire Line
+	7600 1800 7600 3650
+Wire Wire Line
+	8400 2000 8425 2000
+Wire Wire Line
+	8400 2000 8400 2450
+Wire Wire Line
+	8400 2450 9050 2450
+Wire Wire Line
+	9050 2450 9050 1900
+Connection ~ 9050 1900
+Wire Wire Line
+	9050 1900 9025 1900
+Text HLabel 5125 1900 2    50   Input ~ 0
+LM324B
+Wire Wire Line
+	5125 1900 5100 1900
+Connection ~ 5100 1900
 $EndSCHEMATC

Commit message: small fixes in layout. Fabrication files exported.
Parts:
- added C621: 100nF, Capacitor_SMD:C_0805_2012Metric_Pad1.15x1.40mm_HandSolder, symbol Device:C_Small
Connections:
- wire segments 216 -> 219
Other:
- moved on the sheet: C604, C605
Changed lines of the file:
@@
 EESchema Schematic File Version 4
-EELAYER 26 0
+EELAYER 30 0
 EELAYER END
 $Descr A4 11693 8268
@@
 	2700 4750 2650 4750
 Wire Wire Line
-	2650 4750 2650 4850
-Wire Wire Line
 	2650 4850 3100 4850
 $Comp
@@
 	1950 3450 1950 3400
 Wire Wire Line
-	3050 3450 3050 4750
+	3050 3450 3050 4275
 $Comp
 L power:+15V #PWR0615
@@
 L power:+15V #PWR0114
 U 1 1 5DA059B9
-P 2175 4675
-F 0 "#PWR0114" H 2175 4525 50  0001 C CNN
-F 1 "+15V" H 2190 4848 50  0000 C CNN
-F 2 "" H 2175 4675 50  0001 C CNN
-F 3 "" H 2175 4675 50  0001 C CNN
-	1    2175 4675
-	1    0    0    -1
-$EndComp
-Wire Wire Line
-	2075 5025 2175 5025
-Connection ~ 2075 5025
-Wire Wire Line
-	2075 5025 2075 5050
+P 1550 4825
+F 0 "#PWR0114" H 1550 4675 50  0001 C CNN
+F 1 "+15V" H 1565 4998 50  0000 C CNN
+F 2 "" H 1550 4825 50  0001 C CNN
+F 3 "" H 1550 4825 50  0001 C CNN
+	1    1550 4825
+	1    0    0    -1
+$EndComp
+Wire Wire Line
+	2075 5000 2175 5000
+Connection ~ 2075 5000
+Wire Wire Line
+	2075 5000 2075 5025
 $Comp
 L power:GND #PWR0110
 U 1 1 5D4A1ABA
-P 2075 5050
-F 0 "#PWR0110" H 2075 4800 50  0001 C CNN
-F 1 "GND" H 2080 4877 50  0000 C CNN
-F 2 "" H 2075 5050 50  0001 C CNN
-F 3 "" H 2075 5050 50  0001 C CNN
-	1    2075 5050
-	1    0    0    -1
-$EndComp
-Connection ~ 2175 4725
-Wire Wire Line
-	1975 4725 2175 4725
-Wire Wire Line
-	2175 4725 2175 4675
-Wire Wire Line
-	2175 4725 2175 4775
-Wire Wire Line
-	1975 4775 1975 4725
-Wire Wire Line
-	2175 5025 2175 4975
-Wire Wire Line
-	1975 5025 2075 5025
-Wire Wire Line
-	1975 4975 1975 5025
+P 2075 5025
+F 0 "#PWR0110" H 2075 4775 50  0001 C CNN
+F 1 "GND" H 2080 4852 50  0000 C CNN
+F 2 "" H 2075 5025 50  0001 C CNN
+F 3 "" H 2075 5025 50  0001 C CNN
+	1    2075 5025
+	1    0    0    -1
+$EndComp
+Connection ~ 2175 4700
+Wire Wire Line
+	1975 4700 2175 4700
+Wire Wire Line
+	2175 4700 2175 4750
+Wire Wire Line
+	1975 4750 1975 4700
+Wire Wire Line
+	2175 5000 2175 4950
+Wire Wire Line
+	1975 5000 2075 5000
+Wire Wire Line
+	1975 4950 1975 5000
 $Comp
 L Device:C_Small C605
 U 1 1 5D480B54
-P 2175 4875
-F 0 "C605" H 2267 4921 50  0000 L CNN
-F 1 "100nF" H 2267 4830 50  0000 L CNN
-F 2 "Capacitor_SMD:C_0805_2012Metric_Pad1.15x1.40mm_HandSolder" H 2175 4875 50  0001 C CNN
-F 3 "~" H 2175 4875 50  0001 C CNN
-	1    2175 4875
+P 2175 4850
+F 0 "C605" H 2267 4896 50  0000 L CNN
+F 1 "100nF" H 2267 4805 50  0000 L CNN
+F 2 "Capacitor_SMD:C_0805_2012Metric_Pad1.15x1.40mm_HandSolder" H 2175 4850 50  0001 C CNN
+F 3 "~" H 2175 4850 50  0001 C CNN
+	1    2175 4850
 	1    0    0    -1
 $EndComp
@@
 L Device:CP1_Small C?
 U 1 1 5D47B02C
-P 1975 4875
+P 1975 4850
 AR Path="/5AACFFEF/5D47B02C" Ref="C?"  Part="1"
 AR Path="/5D414D87/5D47B02C" Ref="C604"  Part="1"
-F 0 "C604" H 1985 4945 50  0000 L CNN
-F 1 "1uF" H 1985 4795 50  0000 L CNN
-F 2 "Capacitor_Tantalum_SMD:CP_EIA-6032-20_AVX-F_Pad2.25x2.35mm_HandSolder" H 1975 4875 50  0001 C CNN
-F 3 "" H 1975 4875 50  0001 C CNN
-	1    1975 4875
+F 0 "C604" H 1985 4920 50  0000 L CNN
+F 1 "1uF" H 1985 4770 50  0000 L CNN
+F 2 "Capacitor_Tantalum_SMD:CP_EIA-6032-20_AVX-F_Pad2.25x2.35mm_HandSolder" H 1975 4850 50  0001 C CNN
+F 3 "" H 1975 4850 50  0001 C CNN
+	1    1975 4850
 	1    0    0    -1
 $EndComp
@@
 	5125 1900 5100 1900
 Connection ~ 5100 1900
+$Comp
+L power:PWR_FLAG #FLG0102
+U 1 1 5E254110
+P 3050 3450
+F 0 "#FLG0102" H 3050 3525 50  0001 C CNN
+F 1 "PWR_FLAG" H 3075 3675 50  0000 C CNN
+F 2 "" H 3050 3450 50  0001 C CNN
+F 3 "~" H 3050 3450 50  0001 C CNN
+	1    3050 3450
+	1    0    0    -1
+$EndComp
+Connection ~ 3050 3450
+$Comp
+L power:PWR_FLAG #FLG0601
+U 1 1 5E256E60
+P 2650 4550
+F 0 "#FLG0601" H 2650 4625 50  0001 C CNN
+F 1 "PWR_FLAG" H 2675 4775 50  0000 C CNN
+F 2 "" H 2650 4550 50  0001 C CNN
+F 3 "~" H 2650 4550 50  0001 C CNN
+	1    2650 4550
+	1    0    0    -1
+$EndComp
+Wire Wire Line
+	2650 4550 2650 4750
+Connection ~ 2650 4750
+Wire Wire Line
+	2650 4750 2650 4850
+$Comp
+L Device:C_Small C621
+U 1 1 5E28BEFF
+P 1550 4925
+F 0 "C621" H 1642 4971 50  0000 L CNN
+F 1 "100nF" H 1642 4880 50  0000 L CNN
+F 2 "Capacitor_SMD:C_0805_2012Metric_Pad1.15x1.40mm_HandSolder" H 1550 4925 50  0001 C CNN
+F 3 "~" H 1550 4925 50  0001 C CNN
+	1    1550 4925
+	1    0    0    -1
+$EndComp
+$Comp
+L power:GND #PWR0611
+U 1 1 5E28C280
+P 1550 5025
+F 0 "#PWR0611" H 1550 4775 50  0001 C CNN
+F 1 "GND" H 1555 4852 50  0000 C CNN
+F 2 "" H 1550 5025 50  0001 C CNN
+F 3 "" H 1550 5025 50  0001 C CNN
+	1    1550 5025
+	1    0    0    -1
+$EndComp
+Wire Wire Line
+	2175 4275 3050 4275
+Connection ~ 3050 4275
+Wire Wire Line
+	3050 4275 3050 4750
+Wire Wire Line
+	2175 4275 2175 4700
 $EndSCHEMATC

Commit message: driver better referenced to low-side mosfet
Parts:
- removed C621: 100nF, Capacitor_SMD:C_0805_2012Metric_Pad1.15x1.40mm_HandSolder, symbol Device:C_Small
- added C621: 4700uF, Capacitor_THT:CP_Radial_D12.5mm_P5.00mm, symbol Device:CP1_Small
- added D606: ES2A, Diode_SMD:D_MiniMELF_Handsoldering, symbol Diode:LL4148
- added K601: G5LE-1, symbol Relay:G5LE-1
- C602: footprint Capacitor_THT:CP_Radial_D35.0mm_P10.00mm_SnapIn -> Capacitor_THT:CP_Radial_D12.5mm_P5.00mm
Connections:
- net labels added: +12V, ENABLE_RELAY, relay_coil
- net labels removed: +15V, ENABLE
- wire segments 219 -> 229
- no-connect marks 0 -> 1
Other:
- note added: "trazer 18V pra cá"
- moved on the sheet: F601, F602, J611, J612, J613, J614, R611, R612, R613, R614, U603D

Commit message: relay finished
Parts:
- removed R612: 1k, Resistor_SMD:R_0805_2012Metric_Pad1.15x1.40mm_HandSolder, symbol Device:R_Small
- added R1: 90R, Resistor_SMD:R_0805_2012Metric_Pad1.15x1.40mm_HandSolder, symbol Device:R_Small
- K601: footprint (none) -> KicadZeniteSolarLibrary18:Relay_SPDT_SANYOU_SRD_Series_Form_C
Connections:
- net labels added: +18V
- wire segments 229 -> 227
Other:
- note added: "REVIEW RELAY FOOTPRINT\n"
- note removed: "trazer 18V pra cá"
Changed lines of the file:
@@
 $Descr A4 11693 8268
 encoding utf-8
-Sheet 6 7
+Sheet 7 7
 Title ""
 Date ""
@@
 Wire Wire Line
 	2100 2550 2100 2600
-$Comp
-L Device:R_Small R612
-U 1 1 5E1F6547
-P 2450 3150
-F 0 "R612" V 2525 3150 50  0000 C CNN
-F 1 "1k" V 2600 3150 50  0000 C CNN
-F 2 "Resistor_SMD:R_0805_2012Metric_Pad1.15x1.40mm_HandSolder" H 2450 3150 50  0001 C CNN
-F 3 "~" H 2450 3150 50  0001 C CNN
-	1    2450 3150
-	-1   0    0    1
-$EndComp
-Wire Wire Line
-	2450 3250 2450 3300
-Wire Wire Line
-	2450 3300 2100 3300
 Wire Wire Line
 	2100 3300 2100 3250
-Wire Wire Line
-	2450 2350 2450 2300
 Wire Wire Line
 	2075 5000 2175 5000
@@
 	1    0    0    -1
 $EndComp
-Connection ~ 2100 3300
 Wire Wire Line
 	6475 3950 7500 3950
@@
 	1    0    0    -1
 $EndComp
-Wire Wire Line
-	2450 2750 2450 2850
 $Comp
 L power:+12V #PWR0114
@@
 Connection ~ 2175 4275
 Wire Wire Line
-	2675 2850 2450 2850
-Connection ~ 2450 2850
-Wire Wire Line
-	2450 2850 2450 3050
+	2675 3025 2450 3025
 $Comp
 L Relay:G5LE-1 K601
@@
 F 0 "K601" V 9125 3150 50  0000 C CNN
 F 1 "G5LE-1" V 9225 3150 50  0000 C CNN
-F 2 "" H 10200 3100 50  0001 L CNN
+F 2 "KicadZeniteSolarLibrary18:Relay_SPDT_SANYOU_SRD_Series_Form_C" H 10200 3100 50  0001 L CNN
 F 3 "http://www.omron.com/ecb/products/pdf/en-g5le.pdf" H 9750 2750 50  0001 C CNN
 	1    9750 3150
@@
 	10200 2650 10200 2950
 Connection ~ 10200 2950
-Text Label 2675 2850 0    50   ~ 0
+Text Label 2675 3025 0    50   ~ 0
 relay_coil
 Text Label 9250 2950 2    50   ~ 0
@@
 	1    0    0    -1
 $EndComp
-Text Notes 2125 2175 0    50   ~ 0
-trazer 18V pra cá
 $Comp
 L Device:CP1_Small C621
@@
 Wire Wire Line
 	3875 3950 4350 3950
+Text HLabel 2450 2175 0    50   Input ~ 0
++18V
+Wire Wire Line
+	2450 2175 2450 2350
+$Comp
+L Device:R_Small R1
+U 1 1 5E28801E
+P 2450 2900
+F 0 "R1" V 2525 2900 50  0000 C CNN
+F 1 "90R" V 2600 2900 50  0000 C CNN
+F 2 "Resistor_SMD:R_0805_2012Metric_Pad1.15x1.40mm_HandSolder" H 2450 2900 50  0001 C CNN
+F 3 "~" H 2450 2900 50  0001 C CNN
+	1    2450 2900
+	-1   0    0    1
+$EndComp
+Wire Wire Line
+	2450 2800 2450 2750
+Wire Wire Line
+	2450 3025 2450 3000
+Text Notes 9025 3150 0    79   ~ 0
+REVIEW RELAY FOOTPRINT\n
 $EndSCHEMATC

Commit message: Some fixes, ready for heat transfering
Parts:
- added C622, C623, C624, C625, C626, C627: 100n, Capacitor_SMD:C_0805_2012Metric_Pad1.15x1.40mm_HandSolder, symbol Device:C_Small
- added C628: 1uF, Capacitor_Tantalum_SMD:CP_EIA-6032-20_AVX-F_Pad2.25x2.35mm_HandSolder, symbol Device:CP1_Small
- added C629: 100nF, Capacitor_SMD:C_0805_2012Metric_Pad1.15x1.40mm_HandSolder, symbol Device:C_Small
- added D607, D608: LED_RED, LED_SMD:LED_0805_2012Metric_Pad1.15x1.40mm_HandSolder, symbol Device:LED_Small
- added R615: 10R, Resistor_SMD:R_2512_6332Metric, symbol Device:R_Small
- added R616, R618: 330, Resistor_SMD:R_0805_2012Metric_Pad1.15x1.40mm_HandSolder, symbol Device:R_Small
- added R617: 10R, Resistor_SMD:R_2512_6332Metric_Pad1.52x3.35mm_HandSolder, symbol Device:R_Small
- DZ601, DZ602, DZ603, DZ604: value 15V -> 12V
- R601: value 100k -> 50k
- R602, R603: value 1R -> 4R7
- R607, R608: value 1R -> 10R
- renumbered R1 to R612
Connections:
- wire segments 227 -> 278
Other:
- moved on the sheet: C601, C602, C603, C604, C605, C606, C607, C608, C609, C610, C611, C612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
