File: hardware/MCB19_panel.kicad_pcb (KiCad board)
At the start: 2 copper layers, 261.5 x 172.8 mm, 411 parts, among them J401 USART, J402 DISABLE, J601 RJ45, J602 RJ45, J611 +BAT_IN, J612 -BAT_IN, J613 +BAT_OUT, J614 -BAT_OUT, K601 G5LE-1, Q601 IRFP260N, Q602 IRFP260N, Q603 BC857, Q604 BC847, U201 MCP2551-I/SN, U202 MCP2515-xSO, U301 LM7805, U401 ATMEGA328P-PU, U501 LM7812, U601 LM5104MNOPB, U602 INA240A4D, U603 LM324, Y201 16MHz, Y401 16MHz

Commit message: relay pin 1 fixed
Parts:
- removed the C201 at (146.5, 69.1)
- removed the C201 at (56.5, 69.1)
- removed the C202 at (261.2, 51.6)
- removed the C202 at (171.2, 51.6)
- removed the C202 at (81.2, 51.6)
- removed the C203 at (251.4, 64.5)
- removed the C203 at (161.4, 64.5)
- removed the C203 at (71.4, 64.5)
- removed the C204 at (247.6, 62.3)
- removed the C204 at (67.6, 62.3)
- removed the C205 at (263.2, 49.6)
- removed the C205 at (173.2, 49.6)
- removed the C205 at (83.2, 49.6)
- removed the C301 at (208.8, 31.9)
- removed the C301 at (118.8, 31.9)
- removed the C301 at (28.8, 31.9)
- removed the C302 at (207.3, 35.9)
- removed the C302 at (117.3, 35.9)
- removed the C302 at (27.3, 35.9)
- removed the C303 at (215.3, 31.9)
- removed the C303 at (125.3, 31.9)
- removed the C303 at (35.3, 31.9)
- removed the C304 at (213.8, 35.9)
- removed the C304 at (123.8, 35.9)
- removed the C304 at (33.9, 35.9)
- removed the C401 at (252.7, 79.1)
- removed the C401 at (162.7, 79.1)
- removed the C401 at (72.7, 79.1)
- removed the C402 at (251.7, 86.6)
- removed the C402 at (161.7, 86.6)
- removed the C402 at (71.7, 86.6)
- removed the C403 at (245.3, 75.5)
- removed the C403 at (155.3, 75.5)
- removed the C403 at (65.3, 75.5)
- removed the C404 at (249.8, 76.8)
- removed the C404 at (159.8, 76.8)
- removed the C404 at (69.8, 76.8)
- removed the C406 at (270.8, 81.3)
- removed the C406 at (180.8, 81.3)
- removed the C406 at (90.8, 81.3)
- removed the C407 at (255.4, 85.7)
- removed the C407 at (165.4, 85.7)
- removed the C407 at (75.4, 85.7)
- removed the C408 at (257.7, 85.7)
- removed the C408 at (167.7, 85.7)
- removed the C408 at (77.7, 85.7)
- removed the C409 at (259.9, 85.7)
- removed the C409 at (169.9, 85.7)
- removed the C409 at (80.0, 85.7)
- removed the C501 at (208.8, 65.4)
- removed the C501 at (118.8, 65.4)
- removed the C501 at (28.8, 65.4)
- removed the C502 at (207.3, 69.4)
- removed the C502 at (117.3, 69.4)
- removed the C502 at (27.3, 69.4)
- removed the C503 at (215.3, 65.4)
- removed the C503 at (125.3, 65.4)
- removed the C503 at (35.3, 65.4)
- removed the C504 at (213.8, 69.4)
- removed the C504 at (123.8, 69.4)
- removed the C504 at (33.8, 69.4)
- removed the C601 at (231.4, 130.1)
- removed the C601 at (141.4, 130.1)
- removed the C601 at (51.4, 130.1)
- removed the C602 at (214.7, 168.5)
- removed the C602 at (124.7, 168.5)
- removed the C602 at (34.6, 168.5)
- removed the C603 at (230.4, 157.7)
- removed the C603 at (140.4, 157.7)
- removed the C603 at (50.4, 157.7)
- removed the C604 at (224.8, 138.4)
- removed the C604 at (134.8, 138.4)
- removed the C604 at (44.8, 138.4)
- removed the C605 at (229.5, 140.5)
- removed the C605 at (139.5, 140.5)
- removed the C605 at (49.5, 140.5)
- removed the C606 at (220.0, 118.5)
- removed the C606 at (130.0, 118.5)
- removed the C606 at (40.0, 118.5)
- removed the C607 at (238.5, 118.5)
- removed the C607 at (148.5, 118.5)
- removed the C607 at (58.5, 118.5)
- removed the C608 at (243.6, 157.7)
- removed the C608 at (153.6, 157.7)
- removed the C608 at (63.5, 157.7)
- removed the C609 at (243.6, 166.1)
- removed the C609 at (153.6, 166.1)
- removed the C609 at (63.5, 166.1)
- removed the C610 at (230.4, 166.1)
- removed the C610 at (140.4, 166.1)
- removed the C610 at (50.4, 166.1)
- removed the C611 at (247.4, 128.3)
- removed the C611 at (157.4, 128.3)
- removed the C611 at (67.5, 128.3)
- removed the C612 at (266.9, 102.7)
- removed the C612 at (176.9, 102.7)
- removed the C612 at (87.0, 102.7)
- removed the C613 at (216.9, 111.1)
- removed the C613 at (126.9, 111.1)
- removed the C613 at (36.9, 111.1)
- removed the C614 at (214.0, 111.1)
- removed the C614 at (124.0, 111.1)
- removed the C614 at (34.0, 111.1)
- removed the C615 at (219.5, 111.6)
- removed the C615 at (129.5, 111.6)
- removed the C615 at (39.5, 111.6)
- removed the C616 at (221.8, 111.6)
- removed the C616 at (131.8, 111.6)
- removed the C616 at (41.8, 111.6)
- removed the C617 at (235.9, 156.0)
- removed the C617 at (145.9, 156.0)
- removed the C617 at (55.9, 156.0)
- removed the C618 at (233.0, 156.0)
- removed the C618 at (143.0, 156.0)
- removed the C618 at (53.0, 156.0)
- removed the C619 at (240.8, 156.0)
- removed the C619 at (150.8, 156.0)
- removed the C619 at (60.8, 156.0)
- removed the C620 at (238.5, 156.0)
- removed the C620 at (148.5, 156.0)
- removed the C620 at (58.5, 156.0)
- removed the C621 at (214.7, 155.1)
- removed the C621 at (124.7, 155.1)
- removed the C621 at (34.6, 155.1)
- removed the C622 at (226.6, 111.5)
- removed the C622 at (136.6, 111.5)
- removed the C622 at (46.6, 111.5)
- removed the C623 at (224.2, 111.5)
- removed the C623 at (134.2, 111.5)
- removed the C623 at (44.2, 111.5)
- removed the C624 at (229.0, 111.5)
- removed the C624 at (139.0, 111.5)
- removed the C624 at (49.0, 111.5)
- removed the C625 at (231.4, 111.5)
- removed the C625 at (141.4, 111.5)
- removed the C625 at (51.4, 111.5)
- removed the C626 at (233.8, 111.5)
- removed the C626 at (143.8, 111.5)
- removed the C626 at (53.8, 111.5)
- removed the C627 at (236.2, 111.5)
- removed the C627 at (146.2, 111.5)
- removed the C627 at (56.2, 111.5)
- removed the C628 at (271.2, 138.5)
- removed the C628 at (181.2, 138.5)
- removed the C628 at (91.2, 138.5)
- removed the C629 at (267.6, 141.1)
- removed the C629 at (177.6, 141.1)
- removed the C629 at (87.6, 141.1)
- removed the D201 at (234.3, 42.6)
- removed the D201 at (144.3, 42.6)
- removed the D201 at (54.4, 42.6)
- removed the D301 at (206.3, 24.4)
- removed the D301 at (116.3, 24.4)
- removed the D301 at (26.3, 24.4)
- removed the D401 at (273.4, 77.6)
- removed the D401 at (183.4, 77.6)
- removed the D401 at (93.4, 77.6)
- removed the D402 at (260.0, 76.9)
- removed the D402 at (170.0, 76.9)
- removed the D402 at (80.0, 76.9)
- removed the D403 at (235.4, 76.6)
- removed the D403 at (145.4, 76.6)
- removed the D403 at (55.5, 76.6)
- removed the D501 at (203.8, 24.4)
- removed the D501 at (113.8, 24.4)
- removed the D501 at (23.8, 24.4)
- removed the D601 at (227.9, 133.6)
- removed the D601 at (137.9, 133.6)
- removed the D601 at (47.9, 133.6)
- removed the D602 at (236.5, 135.5)
- removed the D602 at (146.5, 135.5)
- removed the D602 at (56.5, 135.5)
- removed the D603 at (218.0, 135.5)
- removed the D603 at (128.0, 135.5)
- removed the D603 at (38.0, 135.5)
- removed the D604 at (216.0, 115.2)
- removed the D604 at (126.0, 115.2)
- removed the D604 at (36.0, 115.2)
- removed the D605 at (234.5, 115.2)
- removed the D605 at (144.5, 115.2)
- removed the D605 at (54.5, 115.2)
- removed the D606 at (256.4, 156.7)
- removed the D606 at (166.4, 156.7)
- removed the D606 at (76.4, 156.7)
- removed the D607 at (272.2, 99.1)
- removed the D607 at (182.2, 99.1)
- removed the D607 at (92.2, 99.1)
- removed the D608 at (255.8, 175.2)
- removed the D608 at (165.8, 175.2)
- removed the D608 at (75.8, 175.2)
- removed the DZ601 at (236.5, 132.5)
- removed the DZ601 at (146.5, 132.5)
- removed the DZ601 at (56.5, 132.5)
- removed the DZ602 at (236.5, 129.5)
- removed the DZ602 at (146.5, 129.5)
- removed the DZ602 at (56.5, 129.5)
- removed the DZ603 at (218.0, 132.5)
- removed the DZ603 at (128.0, 132.5)
- removed the DZ603 at (38.0, 132.5)
- removed the DZ604 at (218.0, 129.5)
- removed the DZ604 at (128.0, 129.5)
- removed the DZ604 at (38.0, 129.5)
- removed the F501 at (210.8, 21.6)
- removed the F501 at (120.8, 21.6)
- removed the F501 at (30.9, 21.6)
- removed the F601 at (205.5, 151.3)
- removed the F601 at (115.5, 151.3)
- removed the F601 at (25.5, 151.3)
- removed the F602 at (270.8, 151.3)
- removed the F602 at (180.8, 151.3)
- removed the F602 at (90.8, 151.3)
- removed the J401 at (259.7, 72.6)
- removed the J401 at (169.7, 72.6)
- removed the J401 at (79.7, 72.6)
- removed the J402 at (234.9, 72.6)
- removed the J402 at (144.9, 72.6)
- removed the J402 at (55.0, 72.6)
- removed the J601 at (231.9, 31.9)
- removed the J601 at (141.9, 31.9)
- removed the J601 at (51.9, 31.9)
- removed the J602 at (252.7, 31.9)
- removed the J602 at (162.7, 31.9)
- removed the J602 at (72.7, 31.9)
- removed the J611 at (210.0, 183.5)
- removed the J611 at (120.0, 183.5)
- removed the J611 at (30.0, 183.5)
- removed the J612 at (229.0, 183.5)
- removed the J612 at (139.0, 183.5)
- removed the J612 at (49.0, 183.5)
- removed the J613 at (266.5, 183.5)
- removed the J613 at (176.5, 183.5)
- removed the J613 at (86.5, 183.5)
- removed the J614 at (248.5, 183.5)
- removed the J614 at (158.5, 183.5)
- removed the J614 at (68.5, 183.5)
- removed the K601 at (258.0, 149.7)
- removed the K601 at (168.0, 149.7)
- removed the K601 at (78.0, 149.7)
- removed the L601 at (236.8, 101.5)
- removed the L601 at (146.8, 101.5)
- removed the L601 at (56.8, 101.5)
- removed the Q601 at (209.0, 124.5)
- removed the Q601 at (119.0, 124.5)
- removed the Q601 at (29.0, 124.5)
- removed the Q602 at (227.5, 124.5)
- removed the Q602 at (137.5, 124.5)
- removed the Q602 at (47.5, 124.5)
- removed the Q603 at (262.6, 141.7)
- removed the Q603 at (172.6, 141.7)
- removed the Q603 at (82.5, 141.7)
- removed the Q604 at (261.6, 137.5)
- removed the Q604 at (171.6, 137.5)
- removed the Q604 at (81.6, 137.5)
- removed the R201 at (265.7, 41.1)
- removed the R201 at (175.7, 41.1)
- removed the R201 at (85.7, 41.1)
- removed the R202 at (269.7, 58.1)
- removed the R202 at (179.7, 58.1)
- removed the R202 at (89.7, 58.1)
- removed the R203 at (261.2, 47.6)
- removed the R203 at (171.2, 47.6)
- removed the R203 at (81.2, 47.6)
- removed the R401 at (270.7, 74.7)
- removed the R401 at (180.7, 74.7)
- removed the R401 at (90.7, 74.7)
- removed the R402 at (265.6, 76.8)
- removed the R402 at (175.6, 76.8)
- removed the R402 at (85.6, 76.8)
- removed the R403 at (263.1, 76.8)
- removed the R403 at (173.1, 76.8)
- removed the R403 at (83.1, 76.8)
- removed the R404 at (257.0, 76.9)
- removed the R404 at (167.0, 76.9)
- removed the R404 at (77.0, 76.9)
- removed the R406 at (237.8, 77.9)
- removed the R406 at (147.8, 77.9)
- removed the R406 at (57.8, 77.9)
- removed the R407 at (255.4, 93.3)
- removed the R407 at (165.4, 93.3)
- removed the R407 at (75.4, 93.3)
- removed the R408 at (257.9, 93.3)
- removed the R408 at (167.9, 93.3)
- removed the R408 at (77.9, 93.3)
- removed the R409 at (260.5, 93.3)
- removed the R409 at (170.5, 93.3)
- removed the R409 at (80.5, 93.3)
- removed the R410 at (240.7, 69.1)
- removed the R410 at (150.7, 69.1)
- removed the R410 at (60.7, 69.1)
- removed the R411 at (268.1, 76.8)
- removed the R411 at (178.2, 76.8)
- removed the R411 at (88.2, 76.8)
- removed the R601 at (235.8, 130.1)
- removed the R601 at (145.8, 130.1)
- removed the R601 at (55.8, 130.1)
- removed the R602 at (229.0, 133.5)
- removed the R602 at (139.0, 133.5)
- removed the R602 at (49.0, 133.5)
- removed the R603 at (210.5, 133.5)
- removed the R603 at (120.5, 133.5)
- removed the R603 at (30.5, 133.5)
- removed the R604 at (229.0, 129.5)
- removed the R604 at (139.0, 129.5)
- removed the R604 at (49.0, 129.5)
- removed the R605 at (210.5, 129.5)
- removed the R605 at (120.5, 129.5)
- removed the R605 at (30.5, 129.5)
- removed the R606 at (245.9, 117.5)
- removed the R606 at (155.9, 117.5)
- removed the R606 at (66.0, 117.5)
- removed the R607 at (213.0, 118.8)
- removed the R607 at (123.0, 118.8)
- removed the R607 at (33.0, 118.8)
- removed the R608 at (231.5, 118.8)
- removed the R608 at (141.5, 118.8)
- removed the R608 at (51.5, 118.8)
- removed the R609 at (251.7, 134.1)
- removed the R609 at (161.7, 134.1)
- removed the R609 at (71.7, 134.1)
- removed the R610 at (247.9, 133.1)
- removed the R610 at (157.9, 133.1)
- removed the R610 at (68.0, 133.1)
- removed the R611 at (265.2, 137.5)
- removed the R611 at (175.2, 137.5)
- removed the R611 at (85.2, 137.5)
- removed the R612 at (262.0, 144.9)
- removed the R612 at (172.0, 144.9)
- removed the R612 at (82.0, 144.9)
- removed the R613 at (210.3, 112.5)
- removed the R613 at (120.3, 112.5)
- removed the R613 at (30.3, 112.5)
- removed the R614 at (210.3, 109.5)
- removed the R614 at (120.3, 109.5)
- removed the R614 at (30.3, 109.5)
- removed the R615 at (213.0, 118.8)
- removed the R615 at (123.0, 118.8)
- removed the R615 at (33.0, 118.8)
- removed the R616 at (270.0, 97.1)
- removed the R616 at (180.0, 97.1)
- removed the R616 at (90.0, 97.1)
- removed the R617 at (231.5, 118.8)
- removed the R617 at (141.5, 118.8)
- removed the R617 at (51.5, 118.8)
- removed the R618 at (256.8, 171.9)
- removed the R618 at (166.8, 171.9)
- removed the R618 at (76.8, 171.9)
- removed the TP201 at (253.2, 43.6)
- removed the TP201 at (163.2, 43.6)
- removed the TP201 at (73.2, 43.6)
- removed the TP202 at (256.2, 43.6)
- removed the TP202 at (166.2, 43.6)
- removed the TP202 at (76.2, 43.6)
- removed the TP203 at (270.2, 64.1)
- removed the TP203 at (180.2, 64.1)
- removed the TP203 at (90.2, 64.1)
- removed the TP204 at (261.2, 64.1)
- removed the TP204 at (171.2, 64.1)
- removed the TP204 at (81.2, 64.1)
- removed the TP205 at (259.2, 43.6)
- removed the TP205 at (169.2, 43.6)
- removed the TP205 at (79.2, 43.6)
- removed the TP206 at (250.2, 43.6)
- removed the TP206 at (160.2, 43.6)
- removed the TP206 at (70.2, 43.6)
- removed the TP207 at (267.2, 44.1)
- removed the TP207 at (177.2, 44.1)
- removed the TP207 at (87.2, 44.1)
- removed the TP208 at (264.2, 44.1)
- removed the TP208 at (174.2, 44.1)
- removed the TP208 at (84.2, 44.1)
- removed the TP209 at (246.2, 51.5)
- removed the TP209 at (156.2, 51.5)
- removed the TP209 at (66.2, 51.5)
- removed the TP401 at (226.0, 87.3)
- removed the TP401 at (136.0, 87.3)
- removed the TP401 at (46.0, 87.3)
- removed the TP402 at (272.0, 93.5)
- removed the TP402 at (182.0, 93.5)
- removed the TP402 at (92.0, 93.5)
- removed the U201 at (265.7, 59.6)
- removed the U201 at (175.7, 59.6)
- removed the U201 at (85.7, 59.6)
- removed the U202 at (253.9, 54.1)
- removed the U202 at (163.9, 54.1)
- removed the U202 at (73.9, 54.1)
- removed the U301 at (208.8, 42.2)
- removed the U301 at (118.8, 42.2)
- removed the U301 at (28.8, 42.2)
- removed the U401 at (268.1, 82.0)
- removed the U401 at (178.2, 82.0)
- removed the U401 at (88.2, 82.0)
- removed the U501 at (208.8, 75.7)
- removed the U501 at (118.8, 75.7)
- removed the U501 at (28.8, 75.7)
- removed the U601 at (233.9, 134.1)
- removed the U601 at (143.9, 134.1)
- removed the U601 at (53.9, 134.1)
- removed the U602 at (245.9, 124.3)
- removed the U602 at (155.9, 124.3)
- removed the U602 at (66.0, 124.3)
- removed the U603 at (265.8, 97.0)
- removed the U603 at (175.8, 97.0)
- removed the U603 at (85.8, 97.0)
- removed the Y201 at (253.9, 64.9)
- removed the Y201 at (163.9, 64.9)
- removed the Y201 at (73.9, 64.9)
- removed the Y401 at (242.8, 75.5)
- removed the Y401 at (152.8, 75.5)
- removed the Y401 at (62.8, 75.5)
- added C201: 100nF, Capacitor_SMD:C_0805_2012Metric_Pad1.15x1.40mm_HandSolder, B.Cu at (237.5, 70.3)
- added C201: 100nF, Capacitor_SMD:C_0805_2012Metric_Pad1.15x1.40mm_HandSolder, B.Cu at (147.5, 70.3)
- added C201: 100nF, Capacitor_SMD:C_0805_2012Metric_Pad1.15x1.40mm_HandSolder, B.Cu at (57.5, 70.3)
- added C202: 100nF, Capacitor_SMD:C_0805_2012Metric_Pad1.15x1.40mm_HandSolder, B.Cu at (262.2, 52.9)
- added C202: 100nF, Capacitor_SMD:C_0805_2012Metric_Pad1.15x1.40mm_HandSolder, B.Cu at (172.2, 52.9)
- added C202: 100nF, Capacitor_SMD:C_0805_2012Metric_Pad1.15x1.40mm_HandSolder, B.Cu at (82.2, 52.9)
- added C203: 22pF, Capacitor_SMD:C_0805_2012Metric_Pad1.15x1.40mm_HandSolder, B.Cu at (252.4, 65.7)
- added C203: 22pF, Capacitor_SMD:C_0805_2012Metric_Pad1.15x1.40mm_HandSolder, B.Cu at (162.4, 65.7)
- added C203: 22pF, Capacitor_SMD:C_0805_2012Metric_Pad1.15x1.40mm_HandSolder, B.Cu at (72.4, 65.7)
- added C204: 22pF, Capacitor_SMD:C_0805_2012Metric_Pad1.15x1.40mm_HandSolder, B.Cu at (248.6, 63.6)
- added C204: 22pF, Capacitor_SMD:C_0805_2012Metric_Pad1.15x1.40mm_HandSolder, B.Cu at (158.6, 63.6)
- added C204: 22pF, Capacitor_SMD:C_0805_2012Metric_Pad1.15x1.40mm_HandSolder, B.Cu at (68.6, 63.6)
- added C205: 100nF, Capacitor_SMD:C_0805_2012Metric_Pad1.15x1.40mm_HandSolder, B.Cu at (264.2, 50.9)
- added C205: 100nF, Capacitor_SMD:C_0805_2012Metric_Pad1.15x1.40mm_HandSolder, B.Cu at (174.2, 50.9)
- added C205: 100nF, Capacitor_SMD:C_0805_2012Metric_Pad1.15x1.40mm_HandSolder, B.Cu at (84.2, 50.9)
- added C301: 1uF, Capacitor_Tantalum_SMD:CP_EIA-6032-20_AVX-F_Pad2.25x2.35mm_HandSolder, B.Cu at (209.8, 33.1)
- added C301: 1uF, Capacitor_Tantalum_SMD:CP_EIA-6032-20_AVX-F_Pad2.25x2.35mm_HandSolder, B.Cu at (119.8, 33.1)
- added C301: 1uF, Capacitor_Tantalum_SMD:CP_EIA-6032-20_AVX-F_Pad2.25x2.35mm_HandSolder, B.Cu at (29.8, 33.1)
- added C302: 100nF, Capacitor_SMD:C_0805_2012Metric_Pad1.15x1.40mm_HandSolder, B.Cu at (208.3, 37.1)
- added C302: 100nF, Capacitor_SMD:C_0805_2012Metric_Pad1.15x1.40mm_HandSolder, B.Cu at (118.3, 37.1)
- added C302: 100nF, Capacitor_SMD:C_0805_2012Metric_Pad1.15x1.40mm_HandSolder, B.Cu at (28.3, 37.1)
- added C303: 100nF, Capacitor_SMD:C_0805_2012Metric_Pad1.15x1.40mm_HandSolder, B.Cu at (216.3, 33.1)
- added C303: 100nF, Capacitor_SMD:C_0805_2012Metric_Pad1.15x1.40mm_HandSolder, B.Cu at (126.3, 33.1)
- added C303: 100nF, Capacitor_SMD:C_0805_2012Metric_Pad1.15x1.40mm_HandSolder, B.Cu at (36.3, 33.1)
- added C304: 1uF, Capacitor_Tantalum_SMD:CP_EIA-6032-20_AVX-F_Pad2.25x2.35mm_HandSolder, B.Cu at (124.8, 37.1)
- added C304: 1uF, Capacitor_Tantalum_SMD:CP_EIA-6032-20_AVX-F_Pad2.25x2.35mm_HandSolder, B.Cu at (34.9, 37.1)
- added C401: 100nF, Capacitor_SMD:C_0805_2012Metric_Pad1.15x1.40mm_HandSolder, B.Cu at (253.7, 80.3)
- added C401: 100nF, Capacitor_SMD:C_0805_2012Metric_Pad1.15x1.40mm_HandSolder, B.Cu at (163.7, 80.3)
- added C401: 100nF, Capacitor_SMD:C_0805_2012Metric_Pad1.15x1.40mm_HandSolder, B.Cu at (73.7, 80.3)
- added C402: 100nF, Capacitor_SMD:C_0805_2012Metric_Pad1.15x1.40mm_HandSolder, B.Cu at (252.7, 87.8)
- added C402: 100nF, Capacitor_SMD:C_0805_2012Metric_Pad1.15x1.40mm_HandSolder, B.Cu at (162.7, 87.8)
- added C402: 100nF, Capacitor_SMD:C_0805_2012Metric_Pad1.15x1.40mm_HandSolder, B.Cu at (72.7, 87.8)
- added C403: 22pF, Capacitor_SMD:C_0805_2012Metric_Pad1.15x1.40mm_HandSolder, B.Cu at (246.3, 76.8)
- added C403: 22pF, Capacitor_SMD:C_0805_2012Metric_Pad1.15x1.40mm_HandSolder, B.Cu at (156.3, 76.8)
- added C403: 22pF, Capacitor_SMD:C_0805_2012Metric_Pad1.15x1.40mm_HandSolder, B.Cu at (66.3, 76.8)
- added C404: 22pF, Capacitor_SMD:C_0805_2012Metric_Pad1.15x1.40mm_HandSolder, B.Cu at (250.8, 78.0)
- added C404: 22pF, Capacitor_SMD:C_0805_2012Metric_Pad1.15x1.40mm_HandSolder, B.Cu at (160.8, 78.0)
- added C404: 22pF, Capacitor_SMD:C_0805_2012Metric_Pad1.15x1.40mm_HandSolder, B.Cu at (70.8, 78.0)
- added C406: 100nF, Capacitor_SMD:C_0805_2012Metric_Pad1.15x1.40mm_HandSolder, B.Cu at (271.8, 82.6)
- added C406: 100nF, Capacitor_SMD:C_0805_2012Metric_Pad1.15x1.40mm_HandSolder, B.Cu at (181.8, 82.6)
- added C406: 100nF, Capacitor_SMD:C_0805_2012Metric_Pad1.15x1.40mm_HandSolder, B.Cu at (91.8, 82.6)
- added C407: 100nF, Capacitor_SMD:C_0805_2012Metric_Pad1.15x1.40mm_HandSolder, B.Cu at (256.4, 87.0)
- added C407: 100nF, Capacitor_SMD:C_0805_2012Metric_Pad1.15x1.40mm_HandSolder, B.Cu at (166.4, 87.0)
- added C407: 100nF, Capacitor_SMD:C_0805_2012Metric_Pad1.15x1.40mm_HandSolder, B.Cu at (76.4, 87.0)
- added C408: 100nF, Capacitor_SMD:C_0805_2012Metric_Pad1.15x1.40mm_HandSolder, B.Cu at (258.7, 87.0)
- added C408: 100nF, Capacitor_SMD:C_0805_2012Metric_Pad1.15x1.40mm_HandSolder, B.Cu at (168.7, 87.0)
- added C408: 100nF, Capacitor_SMD:C_0805_2012Metric_Pad1.15x1.40mm_HandSolder, B.Cu at (78.7, 87.0)
- added C409: 100nF, Capacitor_SMD:C_0805_2012Metric_Pad1.15x1.40mm_HandSolder, B.Cu at (260.9, 87.0)
- added C409: 100nF, Capacitor_SMD:C_0805_2012Metric_Pad1.15x1.40mm_HandSolder, B.Cu at (170.9, 87.0)
- added C409: 100nF, Capacitor_SMD:C_0805_2012Metric_Pad1.15x1.40mm_HandSolder, B.Cu at (81.0, 87.0)
- added C501: 1uF, Capacitor_Tantalum_SMD:CP_EIA-6032-20_AVX-F_Pad2.25x2.35mm_HandSolder, B.Cu at (209.8, 66.7)
- added C501: 1uF, Capacitor_Tantalum_SMD:CP_EIA-6032-20_AVX-F_Pad2.25x2.35mm_HandSolder, B.Cu at (119.8, 66.7)
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Routing:
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
Commit message: some necks removed
Parts:
- removed the C201 at (237.5, 70.3)
- removed the C201 at (147.5, 70.3)
- removed the C201 at (57.5, 70.3)
- removed the C202 at (262.2, 52.9)
- removed the C202 at (172.2, 52.9)
- removed the C202 at (82.2, 52.9)
- removed the C203 at (252.4, 65.7)
- removed the C203 at (162.4, 65.7)
- removed the C203 at (72.4, 65.7)
- removed the C204 at (248.6, 63.6)
- removed the C204 at (158.6, 63.6)
- removed the C204 at (68.6, 63.6)
- removed the C205 at (264.2, 50.9)
- removed the C205 at (174.2, 50.9)
- removed the C205 at (84.2, 50.9)
- removed the C301 at (209.8, 33.1)
- removed the C301 at (119.8, 33.1)
- removed the C301 at (29.8, 33.1)
- removed the C302 at (208.3, 37.1)
- removed the C302 at (118.3, 37.1)
- removed the C302 at (28.3, 37.1)
- removed the C303 at (216.3, 33.1)
- removed the C303 at (126.3, 33.1)
- removed the C303 at (36.3, 33.1)
- removed the C304 at (214.8, 37.1)
- removed the C304 at (124.8, 37.1)
- removed the C304 at (34.9, 37.1)
- removed the C401 at (253.7, 80.3)
- removed the C401 at (163.7, 80.3)
- removed the C401 at (73.7, 80.3)
- removed the C402 at (252.7, 87.8)
- removed the C402 at (162.7, 87.8)
- removed the C402 at (72.7, 87.8)
- removed the C403 at (246.3, 76.8)
- removed the C403 at (156.3, 76.8)
- removed the C403 at (66.3, 76.8)
- removed the C404 at (250.8, 78.0)
- removed the C404 at (160.8, 78.0)
- removed the C404 at (70.8, 78.0)
- removed the C406 at (271.8, 82.6)
- removed the C406 at (181.8, 82.6)
- removed the C406 at (91.8, 82.6)
- removed the C407 at (256.4, 87.0)
- removed the C407 at (166.4, 87.0)
- removed the C407 at (76.4, 87.0)
- removed the C408 at (258.7, 87.0)
- removed the C408 at (168.7, 87.0)
- removed the C408 at (78.7, 87.0)
- removed the C409 at (260.9, 87.0)
- removed the C409 at (170.9, 87.0)
- removed the C409 at (81.0, 87.0)
- removed the C501 at (209.8, 66.7)
- removed the C501 at (119.8, 66.7)
- removed the C501 at (29.8, 66.7)
- removed the C502 at (208.3, 70.7)
- removed the C502 at (118.3, 70.7)
- removed the C502 at (28.3, 70.7)
- removed the C503 at (216.3, 66.7)
- removed the C503 at (126.3, 66.7)
- removed the C503 at (36.3, 66.7)
- removed the C504 at (214.8, 70.7)
- removed the C504 at (124.8, 70.7)
- removed the C504 at (34.8, 70.7)
- removed the C601 at (232.4, 131.3)
- removed the C601 at (142.4, 131.3)
- removed the C601 at (52.4, 131.3)
- removed the C602 at (215.7, 169.8)
- removed the C602 at (125.7, 169.8)
- removed the C602 at (35.6, 169.8)
- removed the C603 at (231.4, 159.0)
- removed the C603 at (141.4, 159.0)
- removed the C603 at (51.4, 159.0)
- removed the C604 at (225.8, 139.7)
- removed the C604 at (135.8, 139.7)
- removed the C604 at (45.8, 139.7)
- removed the C605 at (230.5, 141.8)
- removed the C605 at (140.5, 141.8)
- removed the C605 at (50.5, 141.8)
- removed the C606 at (221.0, 119.8)
- removed the C606 at (131.0, 119.8)
- removed the C606 at (41.0, 119.8)
- removed the C607 at (239.5, 119.8)
- removed the C607 at (149.5, 119.8)
- removed the C607 at (59.5, 119.8)
- removed the C608 at (244.6, 159.0)
- removed the C608 at (154.6, 159.0)
- removed the C608 at (64.5, 159.0)
- removed the C609 at (244.6, 167.3)
- removed the C609 at (154.6, 167.3)
- removed the C609 at (64.5, 167.3)
- removed the C610 at (231.4, 167.3)
- removed the C610 at (141.4, 167.3)
- removed the C610 at (51.4, 167.3)
- removed the C611 at (248.4, 129.6)
- removed the C611 at (158.4, 129.6)
- removed the C611 at (68.5, 129.6)
- removed the C612 at (267.9, 104.0)
- removed the C612 at (177.9, 104.0)
- removed the C612 at (88.0, 104.0)
- removed the C613 at (217.9, 112.3)
- removed the C613 at (127.9, 112.3)
- removed the C613 at (37.9, 112.3)
- removed the C614 at (215.0, 112.3)
- removed the C614 at (125.0, 112.3)
- removed the C614 at (35.0, 112.3)
- removed the C615 at (220.5, 112.9)
- removed the C615 at (130.5, 112.9)
- removed the C615 at (40.5, 112.9)
- removed the C616 at (222.8, 112.9)
- removed the C616 at (132.8, 112.9)
- removed the C616 at (42.8, 112.9)
- removed the C617 at (236.9, 157.2)
- removed the C617 at (146.9, 157.2)
- removed the C617 at (56.9, 157.2)
- removed the C618 at (234.0, 157.2)
- removed the C618 at (144.0, 157.2)
- removed the C618 at (54.0, 157.2)
- removed the C619 at (241.8, 157.3)
- removed the C619 at (151.8, 157.3)
- removed the C619 at (61.8, 157.3)
- removed the C620 at (239.5, 157.3)
- removed the C620 at (149.5, 157.3)
- removed the C620 at (59.5, 157.3)
- removed the C621 at (215.7, 156.3)
- removed the C621 at (125.7, 156.3)
- removed the C621 at (35.6, 156.3)
- removed the C622 at (227.6, 112.8)
- removed the C622 at (137.6, 112.8)
- removed the C622 at (47.6, 112.8)
- removed the C623 at (225.2, 112.8)
- removed the C623 at (135.2, 112.8)
- removed the C623 at (45.2, 112.8)
- removed the C624 at (230.0, 112.8)
- removed the C624 at (140.0, 112.8)
- removed the C624 at (50.0, 112.8)
- removed the C625 at (232.4, 112.8)
- removed the C625 at (142.4, 112.8)
- removed the C625 at (52.4, 112.8)
- removed the C626 at (234.8, 112.8)
- removed the C626 at (144.8, 112.8)
- removed the C626 at (54.8, 112.8)
- removed the C627 at (237.2, 112.8)
- removed the C627 at (147.2, 112.8)
- removed the C627 at (57.2, 112.8)
- removed the C628 at (272.2, 139.8)
- removed the C628 at (182.2, 139.8)
- removed the C628 at (92.2, 139.8)
- removed the C629 at (268.6, 142.3)
- removed the C629 at (178.6, 142.3)
- removed the C629 at (88.6, 142.3)
- removed the D201 at (235.3, 43.9)
- removed the D201 at (145.3, 43.9)
- removed the D201 at (55.4, 43.9)
- removed the D301 at (207.3, 25.6)
- removed the D301 at (117.3, 25.6)
- removed the D301 at (27.3, 25.6)
- removed the D401 at (274.4, 78.8)
- removed the D401 at (184.4, 78.8)
- removed the D401 at (94.4, 78.8)
- removed the D402 at (261.0, 78.2)
- removed the D402 at (171.0, 78.2)
- removed the D402 at (81.0, 78.2)
- removed the D403 at (236.4, 77.8)
- removed the D403 at (146.4, 77.8)
- removed the D403 at (56.5, 77.8)
- removed the D501 at (204.8, 25.6)
- removed the D501 at (114.8, 25.6)
- removed the D501 at (24.8, 25.6)
- removed the D601 at (228.9, 134.8)
- removed the D601 at (138.9, 134.8)
- removed the D601 at (48.9, 134.8)
- removed the D602 at (237.5, 136.8)
- removed the D602 at (147.5, 136.8)
- removed the D602 at (57.5, 136.8)
- removed the D603 at (219.0, 136.8)
- removed the D603 at (129.0, 136.8)
- removed the D603 at (39.0, 136.8)
- removed the D604 at (217.0, 116.5)
- removed the D604 at (127.0, 116.5)
- removed the D604 at (37.0, 116.5)
- removed the D605 at (235.5, 116.5)
- removed the D605 at (145.5, 116.5)
- removed the D605 at (55.5, 116.5)
- removed the D606 at (257.4, 158.2)
- removed the D606 at (167.4, 158.2)
- removed the D606 at (77.4, 158.2)
- removed the D607 at (273.2, 100.3)
- removed the D607 at (183.2, 100.3)
- removed the D607 at (93.2, 100.3)
- removed the D608 at (256.8, 176.5)
- removed the D608 at (166.8, 176.5)
- removed the D608 at (76.8, 176.5)
- removed the DZ601 at (237.5, 133.8)
- removed the DZ601 at (147.5, 133.8)
- removed the DZ601 at (57.5, 133.8)
- removed the DZ602 at (237.5, 130.8)
- removed the DZ602 at (147.5, 130.8)
- removed the DZ602 at (57.5, 130.8)
- removed the DZ603 at (219.0, 133.8)
- removed the DZ603 at (129.0, 133.8)
- removed the DZ603 at (39.0, 133.8)
- removed the DZ604 at (219.0, 130.8)
- removed the DZ604 at (129.0, 130.8)
- removed the DZ604 at (39.0, 130.8)
- removed the F501 at (211.8, 22.8)
- removed the F501 at (121.8, 22.8)
- removed the F501 at (31.9, 22.8)
- removed the F601 at (206.5, 152.6)
- removed the F601 at (116.5, 152.6)
- removed the F601 at (26.5, 152.6)
- removed the F602 at (271.8, 152.6)
- removed the F602 at (181.8, 152.6)
- removed the F602 at (91.8, 152.6)
- removed the J401 at (260.7, 73.8)
- removed the J401 at (170.7, 73.8)
- removed the J401 at (80.7, 73.8)
- removed the J402 at (235.9, 73.8)
- removed the J402 at (145.9, 73.8)
- removed the J402 at (56.0, 73.8)
- removed the J601 at (232.9, 33.1)
- removed the J601 at (142.9, 33.1)
- removed the J601 at (52.9, 33.1)
- removed the J602 at (253.7, 33.1)
- removed the J602 at (163.7, 33.1)
- removed the J602 at (73.7, 33.1)
- removed the J611 at (211.0, 184.8)
- removed the J611 at (121.0, 184.8)
- removed the J611 at (31.0, 184.8)
- removed the J612 at (230.0, 184.8)
- removed the J612 at (140.0, 184.8)
- removed the J612 at (50.0, 184.8)
- removed the J613 at (267.5, 184.8)
- removed the J613 at (177.5, 184.8)
- removed the J613 at (87.5, 184.8)
- removed the J614 at (249.5, 184.8)
- removed the J614 at (159.5, 184.8)
- removed the J614 at (69.5, 184.8)
- removed the K601 at (259.0, 150.9)
- removed the K601 at (169.0, 150.9)
- removed the K601 at (79.0, 150.9)
- removed the L601 at (237.8, 102.8)
- removed the L601 at (147.8, 102.8)
- removed the L601 at (57.8, 102.8)
- removed the Q601 at (210.0, 125.8)
- removed the Q601 at (120.0, 125.8)
- removed the Q601 at (30.0, 125.8)
- removed the Q602 at (228.5, 125.8)
- removed the Q602 at (138.5, 125.8)
- removed the Q602 at (48.5, 125.8)
- removed the Q603 at (263.6, 142.9)
- removed the Q603 at (173.6, 142.9)
- removed the Q603 at (83.5, 142.9)
- removed the Q604 at (262.6, 138.8)
- removed the Q604 at (172.6, 138.8)
- removed the Q604 at (82.6, 138.8)
- removed the R201 at (266.7, 42.4)
- removed the R201 at (176.7, 42.4)
- removed the R201 at (86.7, 42.4)
- removed the R202 at (270.7, 59.4)
- removed the R202 at (180.7, 59.4)
- removed the R202 at (90.7, 59.4)
- removed the R203 at (262.2, 48.9)
- removed the R203 at (172.2, 48.9)
- removed the R203 at (82.2, 48.9)
- removed the R401 at (271.7, 75.9)
- removed the R401 at (181.7, 75.9)
- removed the R401 at (91.7, 75.9)
- removed the R402 at (266.6, 78.0)
- removed the R402 at (176.6, 78.0)
- removed the R402 at (86.6, 78.0)
- removed the R403 at (264.1, 78.0)
- removed the R403 at (174.1, 78.0)
- removed the R403 at (84.1, 78.0)
- removed the R404 at (258.0, 78.2)
- removed the R404 at (168.0, 78.2)
- removed the R404 at (78.0, 78.2)
- removed the R406 at (238.8, 79.2)
- removed the R406 at (148.8, 79.2)
- removed the R406 at (58.8, 79.2)
- removed the R407 at (256.4, 94.6)
- removed the R407 at (166.4, 94.6)
- removed the R407 at (76.4, 94.6)
- removed the R408 at (258.9, 94.6)
- removed the R408 at (168.9, 94.6)
- removed the R408 at (78.9, 94.6)
- removed the R409 at (261.5, 94.6)
- removed the R409 at (171.5, 94.6)
- removed the R409 at (81.5, 94.6)
- removed the R410 at (241.7, 70.3)
- removed the R410 at (151.7, 70.3)
- removed the R410 at (61.7, 70.3)
- removed the R411 at (269.1, 78.0)
- removed the R411 at (179.2, 78.0)
- removed the R411 at (89.2, 78.0)
- removed the R601 at (236.8, 131.3)
- removed the R601 at (146.8, 131.3)
- removed the R601 at (56.8, 131.3)
- removed the R602 at (230.0, 134.8)
- removed the R602 at (140.0, 134.8)
- removed the R602 at (50.0, 134.8)
- removed the R603 at (211.5, 134.8)
- removed the R603 at (121.5, 134.8)
- removed the R603 at (31.5, 134.8)
- removed the R604 at (230.0, 130.8)
- removed the R604 at (140.0, 130.8)
- removed the R604 at (50.0, 130.8)
- removed the R605 at (211.5, 130.8)
- removed the R605 at (121.5, 130.8)
- removed the R605 at (31.5, 130.8)
- removed the R606 at (246.9, 118.8)
- removed the R606 at (156.9, 118.8)
- removed the R606 at (67.0, 118.8)
- removed the R607 at (214.0, 120.0)
- removed the R607 at (124.0, 120.0)
- removed the R607 at (34.0, 120.0)
- removed the R608 at (232.5, 120.0)
- removed the R608 at (142.5, 120.0)
- removed the R608 at (52.5, 120.0)
- removed the R609 at (252.7, 135.3)
- removed the R609 at (162.7, 135.3)
- removed the R609 at (72.7, 135.3)
- removed the R610 at (248.9, 134.3)
- removed the R610 at (158.9, 134.3)
- removed the R610 at (69.0, 134.3)
- removed the R611 at (266.2, 138.8)
- removed the R611 at (176.2, 138.8)
- removed the R611 at (86.2, 138.8)
- removed the R612 at (263.0, 146.2)
- removed the R612 at (173.0, 146.2)
- removed the R612 at (83.0, 146.2)
- removed the R613 at (211.3, 113.8)
- removed the R613 at (121.3, 113.8)
- removed the R613 at (31.3, 113.8)
- removed the R614 at (211.3, 110.8)
- removed the R614 at (121.3, 110.8)
- removed the R614 at (31.3, 110.8)
- removed the R615 at (214.0, 120.0)
- removed the R615 at (124.0, 120.0)
- removed the R615 at (34.0, 120.0)
- removed the R616 at (271.0, 98.3)
- removed the R616 at (181.0, 98.3)
- removed the R616 at (91.0, 98.3)
- removed the R617 at (232.5, 120.0)
- removed the R617 at (142.5, 120.0)
- removed the R617 at (52.5, 120.0)
- removed the R618 at (257.8, 173.2)
- removed the R618 at (167.8, 173.2)
- removed the R618 at (77.8, 173.2)
- removed the TP201 at (254.2, 44.9)
- removed the TP201 at (164.2, 44.9)
- removed the TP201 at (74.2, 44.9)
- removed the TP202 at (257.2, 44.9)
- removed the TP202 at (167.2, 44.9)
- removed the TP202 at (77.2, 44.9)
- removed the TP203 at (271.2, 65.3)
- removed the TP203 at (181.2, 65.3)
- removed the TP203 at (91.2, 65.3)
- removed the TP204 at (262.2, 65.3)
- removed the TP204 at (172.2, 65.3)
- removed the TP204 at (82.2, 65.3)
- removed the TP205 at (260.2, 44.9)
- removed the TP205 at (170.2, 44.9)
- removed the TP205 at (80.2, 44.9)
- removed the TP206 at (251.2, 44.9)
- removed the TP206 at (161.2, 44.9)
- removed the TP206 at (71.2, 44.9)
- removed the TP207 at (268.2, 45.4)
- removed the TP207 at (178.2, 45.4)
- removed the TP207 at (88.2, 45.4)
- removed the TP208 at (265.2, 45.4)
- removed the TP208 at (175.2, 45.4)
- removed the TP208 at (85.2, 45.4)
- removed the TP209 at (247.2, 52.7)
- removed the TP209 at (157.2, 52.7)
- removed the TP209 at (67.2, 52.7)
- removed the TP401 at (227.0, 88.5)
- removed the TP401 at (137.0, 88.5)
- removed the TP401 at (47.0, 88.5)
- removed the TP402 at (273.0, 94.8)
- removed the TP402 at (183.0, 94.8)
- removed the TP402 at (93.0, 94.8)
- removed the U201 at (266.7, 60.9)
- removed the U201 at (176.7, 60.9)
- removed the U201 at (86.7, 60.9)
- removed the U202 at (254.9, 55.3)
- removed the U202 at (164.9, 55.3)
- removed the U202 at (74.9, 55.3)
- removed the U301 at (209.8, 43.5)
- removed the U301 at (119.8, 43.5)
- removed the U301 at (29.8, 43.5)
- removed the U401 at (269.1, 83.2)
- removed the U401 at (179.2, 83.2)
- removed the U401 at (89.2, 83.2)
- removed the U501 at (209.8, 77.0)
- removed the U501 at (119.8, 77.0)
- removed the U501 at (29.8, 77.0)
- removed the U601 at (234.9, 135.3)
- removed the U601 at (144.9, 135.3)
- removed the U601 at (54.9, 135.3)
- removed the U602 at (246.9, 125.5)
- removed the U602 at (156.9, 125.5)
- removed the U602 at (67.0, 125.5)
- removed the U603 at (266.8, 98.2)
- removed the U603 at (176.8, 98.2)
- removed the U603 at (86.8, 98.2)
- removed the Y201 at (254.9, 66.1)
- removed the Y201 at (164.9, 66.1)
- removed the Y201 at (74.9, 66.1)
- removed the Y401 at (243.8, 76.8)
- removed the Y401 at (153.8, 76.8)
- removed the Y401 at (63.8, 76.8)
- added C201: 100nF, Capacitor_SMD:C_0805_2012Metric_Pad1.15x1.40mm_HandSolder, B.Cu at (234.0, 69.1)
- added C201: 100nF, Capacitor_SMD:C_0805_2012Metric_Pad1.15x1.40mm_HandSolder, B.Cu at (146.5, 69.1)
- added C201: 100nF, Capacitor_SMD:C_0805_2012Metric_Pad1.15x1.40mm_HandSolder, B.Cu at (59.0, 69.1)
- added C202: 100nF, Capacitor_SMD:C_0805_2012Metric_Pad1.15x1.40mm_HandSolder, B.Cu at (258.7, 51.6)
- added C202: 100nF, Capacitor_SMD:C_0805_2012Metric_Pad1.15x1.40mm_HandSolder, B.Cu at (171.2, 51.6)
- added C202: 100nF, Capacitor_SMD:C_0805_2012Metric_Pad1.15x1.40mm_HandSolder, B.Cu at (83.7, 51.6)
- added C203: 22pF, Capacitor_SMD:C_0805_2012Metric_Pad1.15x1.40mm_HandSolder, B.Cu at (248.9, 64.5)
- added C203: 22pF, Capacitor_SMD:C_0805_2012Metric_Pad1.15x1.40mm_HandSolder, B.Cu at (161.4, 64.5)
- added C203: 22pF, Capacitor_SMD:C_0805_2012Metric_Pad1.15x1.40mm_HandSolder, B.Cu at (73.9, 64.5)
- added C204: 22pF, Capacitor_SMD:C_0805_2012Metric_Pad1.15x1.40mm_HandSolder, B.Cu at (245.1, 62.3)
- added C204: 22pF, Capacitor_SMD:C_0805_2012Metric_Pad1.15x1.40mm_HandSolder, B.Cu at (157.6, 62.3)
- added C204: 22pF, Capacitor_SMD:C_0805_2012Metric_Pad1.15x1.40mm_HandSolder, B.Cu at (70.1, 62.3)
- added C205: 100nF, Capacitor_SMD:C_0805_2012Metric_Pad1.15x1.40mm_HandSolder, B.Cu at (260.7, 49.6)
- added C205: 100nF, Capacitor_SMD:C_0805_2012Metric_Pad1.15x1.40mm_HandSolder, B.Cu at (173.2, 49.6)
- added C205: 100nF, Capacitor_SMD:C_0805_2012Metric_Pad1.15x1.40mm_HandSolder, B.Cu at (85.7, 49.6)
- added C301: 1uF, Capacitor_Tantalum_SMD:CP_EIA-6032-20_AVX-F_Pad2.25x2.35mm_HandSolder, B.Cu at (206.2, 31.9)
- added C301: 1uF, Capacitor_Tantalum_SMD:CP_EIA-6032-20_AVX-F_Pad2.25x2.35mm_HandSolder, B.Cu at (118.8, 31.9)
- added C301: 1uF, Capacitor_Tantalum_SMD:CP_EIA-6032-20_AVX-F_Pad2.25x2.35mm_HandSolder, B.Cu at (31.2, 31.9)
- added C302: 100nF, Capacitor_SMD:C_0805_2012Metric_Pad1.15x1.40mm_HandSolder, B.Cu at (204.8, 35.9)
- added C302: 100nF, Capacitor_SMD:C_0805_2012Metric_Pad1.15x1.40mm_HandSolder, B.Cu at (117.3, 35.9)
- added C302: 100nF, Capacitor_SMD:C_0805_2012Metric_Pad1.15x1.40mm_HandSolder, B.Cu at (29.8, 35.9)
- added C303: 100nF, Capacitor_SMD:C_0805_2012Metric_Pad1.15x1.40mm_HandSolder, B.Cu at (212.8, 31.9)
- added C303: 100nF, Capacitor_SMD:C_0805_2012Metric_Pad1.15x1.40mm_HandSolder, B.Cu at (125.3, 31.9)
- added C303: 100nF, Capacitor_SMD:C_0805_2012Metric_Pad1.15x1.40mm_HandSolder, B.Cu at (37.8, 31.9)
- added C304: 1uF, Capacitor_Tantalum_SMD:CP_EIA-6032-20_AVX-F_Pad2.25x2.35mm_HandSolder, B.Cu at (211.3, 35.9)
- added C304: 1uF, Capacitor_Tantalum_SMD:CP_EIA-6032-20_AVX-F_Pad2.25x2.35mm_HandSolder, B.Cu at (123.8, 35.9)
- added C304: 1uF, Capacitor_Tantalum_SMD:CP_EIA-6032-20_AVX-F_Pad2.25x2.35mm_HandSolder, B.Cu at (36.4, 35.9)
- added C401: 100nF, Capacitor_SMD:C_0805_2012Metric_Pad1.15x1.40mm_HandSolder, B.Cu at (250.2, 79.1)
- added C401: 100nF, Capacitor_SMD:C_0805_2012Metric_Pad1.15x1.40mm_HandSolder, B.Cu at (162.7, 79.1)
- added C401: 100nF, Capacitor_SMD:C_0805_2012Metric_Pad1.15x1.40mm_HandSolder, B.Cu at (75.2, 79.1)
- added C402: 100nF, Capacitor_SMD:C_0805_2012Metric_Pad1.15x1.40mm_HandSolder, B.Cu at (249.2, 86.6)
- added C402: 100nF, Capacitor_SMD:C_0805_2012Metric_Pad1.15x1.40mm_HandSolder, B.Cu at (161.7, 86.6)
- added C402: 100nF, Capacitor_SMD:C_0805_2012Metric_Pad1.15x1.40mm_HandSolder, B.Cu at (74.2, 86.6)
- added C403: 22pF, Capacitor_SMD:C_0805_2012Metric_Pad1.15x1.40mm_HandSolder, B.Cu at (242.8, 75.5)
- added C403: 22pF, Capacitor_SMD:C_0805_2012Metric_Pad1.15x1.40mm_HandSolder, B.Cu at (155.3, 75.5)
- added C403: 22pF, Capacitor_SMD:C_0805_2012Metric_Pad1.15x1.40mm_HandSolder, B.Cu at (67.8, 75.5)
- added C404: 22pF, Capacitor_SMD:C_0805_2012Metric_Pad1.15x1.40mm_HandSolder, B.Cu at (247.3, 76.8)
- added C404: 22pF, Capacitor_SMD:C_0805_2012Metric_Pad1.15x1.40mm_HandSolder, B.Cu at (159.8, 76.8)
- added C404: 22pF, Capacitor_SMD:C_0805_2012Metric_Pad1.15x1.40mm_HandSolder, B.Cu at (72.3, 76.8)
- added C406: 100nF, Capacitor_SMD:C_0805_2012Metric_Pad1.15x1.40mm_HandSolder, B.Cu at (268.2, 81.3)
- added C406: 100nF, Capacitor_SMD:C_0805_2012Metric_Pad1.15x1.40mm_HandSolder, B.Cu at (180.8, 81.3)
- added C406: 100nF, Capacitor_SMD:C_0805_2012Metric_Pad1.15x1.40mm_HandSolder, B.Cu at (93.2, 81.3)
- added C407: 100nF, Capacitor_SMD:C_0805_2012Metric_Pad1.15x1.40mm_HandSolder, B.Cu at (252.9, 85.7)
- added C407: 100nF, Capacitor_SMD:C_0805_2012Metric_Pad1.15x1.40mm_HandSolder, B.Cu at (165.4, 85.7)
- added C407: 100nF, Capacitor_SMD:C_0805_2012Metric_Pad1.15x1.40mm_HandSolder, B.Cu at (77.9, 85.7)
- added C408: 100nF, Capacitor_SMD:C_0805_2012Metric_Pad1.15x1.40mm_HandSolder, B.Cu at (255.2, 85.7)
- added C408: 100nF, Capacitor_SMD:C_0805_2012Metric_Pad1.15x1.40mm_HandSolder, B.Cu at (167.7, 85.7)
- added C408: 100nF, Capacitor_SMD:C_0805_2012Metric_Pad1.15x1.40mm_HandSolder, B.Cu at (80.2, 85.7)
- added C409: 100nF, Capacitor_SMD:C_0805_2012Metric_Pad1.15x1.40mm_HandSolder, B.Cu at (257.4, 85.7)
- added C409: 100nF, Capacitor_SMD:C_0805_2012Metric_Pad1.15x1.40mm_HandSolder, B.Cu at (169.9, 85.7)
- added C409: 100nF, Capacitor_SMD:C_0805_2012Metric_Pad1.15x1.40mm_HandSolder, B.Cu at (82.5, 85.7)
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Routing:
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Other:
- board size 261.5 x 172.8 mm -> 256.5 x 172.8 mm

Commit message: references added to pdf
Routing:
- net (no net): vias 88 -> 1088
Other:
- rule via_min_drill: 0.3 -> 0.03
- rule via_min_size: 0.4 -> 0.04
