File: hardware/supplies.kicad_sch (KiCad schematic)
At the start: 6 parts, among them U301 LM7805

Commit message: Schematic organization improvement, use <driver> sheet as example
Parts:
- renumbered C301 to C302
Changed lines of the file:
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@@
 (kicad_sch
-	(version 20231120)
+	(version 20250114)
 	(generator "eeschema")
-	(generator_version "8.0")
+	(generator_version "9.0")
 	(paper "A4")
 	(junction
@@
 		(on_board yes)
 		(dnp no)
-		(property "Reference" "C301"
+		(property "Reference" "C302"
 			(at 147.574 99.822 0)
 			(effects
@@
 		(on_board yes)
 		(dnp no)
-		(property "Reference" "#FLG0101"
+		(property "Reference" "#FLG0501"
 			(at 147.32 74.295 0)
 			(effects
