File: hardware/driver.kicad_sch (KiCad schematic)
At the start: 74 parts, among them J611 +BAT_IN, J612 -BAT_IN, J613 +BAT_OUT, J614 -BAT_OUT, K601 G5LE-1, Q601 IRFP260N, Q602 IRFP260N, Q603 BC857, Q604 BC847, U601 LM5104MNOPB, U602 INA240A4D, U603 LM324

Commit message: Schematic organization improvement, use <driver> sheet as example
Parts:
- C602, C604, C621, C628: symbol Device:CP1_Small -> Device:C_Polarized
Connections:
- net +12V: now also C604.1
- net +18V: now also C628.1
- net +BATT: now also C602.1, C602.2, C603.2, C604.2, C605.2, C607.2, C608.2, C609.2, C610.2, C611.1, C612.1, C613.2, C614.2, C615.2, C616.2, C617.2, C618.2, C619.2, C620.2, C621.1, C621.2, C622.2, C623.2, C624.2, C625.2, C626.2, C627.2, C628.2, C629.2, D606.2 (A), D607.1 (K), D608.1 (K), DZ602.2 (A), J612.1 (Pin_1), J614.1 (Pin_1), K601.5, Q602.3 (S), R601.2, R604.1, R610.1, R611.1, U601.7 (VSS), U602.2 (GND), U602.3 (REF2), U602.4 (GND), U602.7 (REF1), U603.10 (+), U603.11 (V-), U603.12 (+)
- net Shunt-: now reaches L601.1, R606.1, U602.1 (-)
- net HIGH_SOURCE: now reaches C601.2, C606.2, D605.2 (A), DZ604.2 (A), Q601.3 (S), Q602.2 (D), Q602.4 (D), R605.1, R606.2, R608.2, R617.2, U601.4 (HS), U602.8 (+)
- net GATE_LS: now reaches D602.2 (A), DZ601.2 (A), Q602.1 (G), R602.1, R604.2
- net GATE_HS: now reaches D603.2 (A), DZ603.2 (A), Q601.1 (G), R603.1, R605.2
- net bat_out_+: now reaches F602.1, K601.3, R618.1
- net bat_out_+: no longer R609.2
- removed net GND: C603.2, C605.2, C607.2, C608.2, C609.2, C610.2, C611.1, C612.1, C613.2, C614.2, C615.2, C616.2, C617.2, C618.2, C619.2, C620.2, C622.2, C623.2, C624.2, C625.2, C626.2, C627.2, C629.2, D606.2 (A), D607.1 (K), D608.1 (K), DZ602.2 (A), J612.1 (Pin_1), J614.1 (Pin_1), K601.5, Q602.3 (S), R601.2, R604.1, R610.1, R611.1, R614.1, U601.7 (VSS), U602.2 (GND), U602.3 (REF2), U602.4 (GND), U602.7 (REF1), U603.10 (+), U603.11 (V-), U603.12 (+)
- new net bat_in_-: R614.1
- new net bat_out+: R609.2
Other:
- note added: "ANALOG"
- note added: "BUCK CONVERTER"
- note added: "DRIVER"
- note added: "MISSING PROTECTIONS"
- note added: "RELAY ACTIVATION"
- moved on the sheet: C601, C603, C605, C606, C607, C608, C609, C610, C611, C612, C613, C614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

Commit message: add diode protections for Vsense OpAmps and uC port
Parts:
- added D1, D2: Zener 5V1, Diode_SMD:D_MiniMELF, symbol Diode:BZV55B5V1
- added D4, D5: BAT54J, Diode_SMD:D_SOD-323F, symbol Diode:BAT54J
Connections:
- net +BATT: now also D1.2 (A), D2.2 (A), D4.2 (A), D5.2 (A)
- net at R609.1, R610.2, U603.3 (+): now also D2.1 (K), D5.1 (K)
- net at R613.1, R614.2, U603.5 (+): now also D1.1 (K), D4.1 (K)
Other:
- note removed: "MISSING PROTECTIONS"
- moved on the sheet: R609, R610, R613, R614, U603A, U603B, U603C, U603D
